File: board_sr/sr_controller_v0/sr_controller_v0.brd (EAGLE design)
At the start: 65 x 56 mm, 73 parts, among them K1 PIN20X2, Q1 32kHz, Q3 IRF5210

Commit message: Update schematic
Parts:
- removed CN1: (no value), microbuilder:USB_HOST-PTH
- added R28: R10K, resistor:R0805
- added R29: R2K, resistor:R0805
- added U$8: 74HC4053D, tigorcustom:SO16
- V_SENSORS: device con-ptr500:AK300/4 -> con-ptr500:AK300/5
- moved T4 431.0 mm to (39.0, -62.0), turned to 270 degrees
- moved R17 220.7 mm to (38.0, -86.0), turned to 270 degrees
- moved R16 219.2 mm to (38.0, -82.0), turned to 270 degrees
- moved R15 215.8 mm to (43.0, -86.0), turned to 270 degrees
- moved R14 214.4 mm to (43.0, -82.0), turned to 270 degrees
- moved C6 206.8 mm to (62.0, -56.0), turned to 270 degrees
- moved C5 206.2 mm to (62.0, -52.0), turned to 90 degrees
- moved C4 202.2 mm to (74.0, -26.0), turned to 90 degrees
- moved C3 201.7 mm to (74.0, -22.0), turned to 90 degrees
- moved R4 198.7 mm to (48.0, 85.0), turned to 270 degrees
- moved U$4 196.8 mm to (57.0, -54.0), turned to 270 degrees
- moved R8 192.8 mm to (63.0, -7.00), turned to 270 degrees
- moved U$2 192.8 mm to (69.0, -24.0), turned to 270 degrees
- moved V_SENSORS 192.1 mm to (-61.0, -381.0)
- moved R7 187.6 mm to (61.0, -7.00), turned to 90 degrees
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Connections:
- removed net N$17 (its old number): R16.1, V_SENSORS.4
- new net N$19: R28.1, V_SENSORS.4
- new net N$20: R16.1, V_SENSORS.5
- new net N$34: R15.2
- new net SELECT_SENSOR: U$1.13, U$8.11
- new net SENSOR_HI_1: R14.2, R15.1, U$8.13
- new net SENSOR_HI_2: R28.2, R29.1, U$8.12
- net +3V3: no longer K1.1, K1.17
- net +5V: now also U$8.16; no longer CN1.VBUS
- net GND: now also R29.2, U$8.6, U$8.7, U$8.8; no longer CN1.GND, R15.2
- net SENSOR_HUG_IDIR: now also U$8.14; no longer R14.2, R15.1
Other:
- outline, holes or cut-outs redrawn

Commit message: Update PCB design
Parts:
- removed B1: RECTIFIER-RB1A, rectifier:RB1A
- removed C2: C470uF, resistor:E2-5
- removed D1: 5.1V, diode:ZDIO-7.5
- removed OK1: PC817, optocoupler:DIL04
- removed R2: R470R, resistor:0207/10
- removed R3: R270R, resistor:M0805
- removed R4: R10K, resistor:R0805
- added C14: C100N, resistor:C0805K
- added R30: R1K, resistor:R0805
- added R31: R2K, resistor:R0805
- added R32: R100K, resistor:0309V
- added R33: R2K, resistor:0309V
- added U$9: TRANSFORMER, bontor:TV16
- R11: value R1K -> R2K
- R13: value R2K -> R1K
- moved R28 529.4 mm to (48.8, 14.5), flipped to the bottom
- moved R29 524.6 mm to (44.8, 14.5), flipped to the bottom
- moved U$8 484.2 mm to (36.2, 13.2), flipped to the bottom, turned to 90 degrees
- moved U$7 471.1 mm to (34.0, 2.00), turned to 90 degrees
- moved U$6 464.2 mm to (51.5, 2.00), turned to 90 degrees
- moved LED2 461.7 mm to (-19.5, 66.2)
- moved T2 459.6 mm to (-22.0, 66.5)
- moved R27 454.6 mm to (-31.0, 52.0), turned to 180 degrees
- moved R24 450.0 mm to (-23.5, 62.2), turned to 90 degrees
- moved R26 449.3 mm to (-19.5, 62.2), turned to 90 degrees
- moved T3 447.1 mm to (-31.0, 49.0), turned to 180 degrees
- moved R25 445.2 mm to (-21.5, 62.2), turned to 270 degrees
- moved R23 432.7 mm to (-36.8, 60.8), turned to 90 degrees
- moved LED1 431.7 mm to (-37.0, 64.8)
- moved R22 426.5 mm to (-32.2, 60.8), turned to 270 degrees
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Connections:
- removed net N$17: R10.1, V_SENSORS.1
- removed net N$34: R15.2
- removed net N$7: B1.+, C2.+, D1.C, OK1.1
- removed net N$8: B1.-, C2.-, D1.A, R3.1
- removed net N$9: OK1.2, R3.2
- new net N$35: R30.1, U$1.1
- new net N$36: R32.2, U$9.IA
- new net N$38: C14.2, R33.1, U$9.OB
- net +5V: no longer R4.1
- net AGND: now also C14.1
- net ARDU_TX: now also R30.2, R31.1; no longer U$1.1
- net CTRL_CHARGING: now also K1.11; no longer K1.12
- net CTRL_SIM_PWRKEY: now also K1.15
- net DHT_DATA: now also U$1.13; no longer U$1.15
- net GND: now also R15.2, R31.2, V_ACCU.1, V_LOAD.1, V_PWR_SPLY.1; no longer OK1.3, V_ACCU.2, V_LOAD.2, V_PWR_SPLY.2
- net N$1: now also R32.1, VAC.2; no longer B1.AC1, VAC.1
- net N$12: now also V_PWR_SPLY.2; no longer V_PWR_SPLY.1
- net N$2: now also U$9.IB, VAC.1; no longer R2.1, VAC.2
- net N$6: now also R12.1, V_SENSORS.2; no longer B1.AC2, R2.2
- net SELECT_SENSOR: now also U$1.9; no longer U$1.13
- net SENSOR_BUC: now also R12.2, R13.1, U$1.28; no longer R10.2, R11.1, U$1.25
- net SENSOR_HUG_IDIR: now also U$1.26; no longer U$1.28
- net SENSOR_SCADA: now also U$1.25; no longer U$1.27
- net SENSOR_SCPC: now also R10.2, R11.1, U$1.27; no longer R12.2, R13.1, U$1.26
- net SENSOR_VAC: now also R33.2, U$9.OA; no longer OK1.4, R4.2
- net USIM_DATA: now also D3.1; no longer D3.3
- net USIM_RST: now also D3.3; no longer D3.5
- net USIM_VDD: now also D3.5; no longer D3.1
- net VBAT: now also V_ACCU.2; no longer V_ACCU.1
- net VIN: now also R10.1, V_SENSORS.1; no longer R12.1, V_SENSORS.2
- net VLOAD: now also V_LOAD.2; no longer V_LOAD.1
Routing:
- net GND: track 0.00 -> 149.6 mm
- net SENSOR_SCPC: track 0.00 -> 45.7 mm, vias 0 -> 1
- net +5V: track 0.00 -> 45.4 mm
- net SENSOR_HUG_IDIR: track 0.00 -> 39.9 mm, vias 0 -> 1
- net SENSOR_BUC: track 0.00 -> 38.9 mm, vias 0 -> 1
- net VIN: track 0.00 -> 35.5 mm
- net SENSOR_SCADA: track 0.00 -> 26.3 mm, vias 0 -> 1
- net SELECT_SENSOR: track 0.00 -> 21.0 mm, vias 0 -> 1
- net N$20: track 0.00 -> 16.7 mm
- net N$2: track 0.00 -> 16.1 mm
- net N$19: track 0.00 -> 14.9 mm
- net N$22: track 0.00 -> 14.1 mm, vias 0 -> 1
- net DHT_DATA: track 0.00 -> 13.9 mm
- net N$18: track 0.00 -> 12.7 mm
- net N$38: track 0.00 -> 11.5 mm
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Other:
- board size 65 x 56 mm -> 125 x 56 mm
