File: board_sr/sr_controller_v0/sr_controller_v0.sch (EAGLE design)
At the start: 73 parts, among them K1 PIN20X2, Q1 32kHz, Q3 IRF5210

Commit message: Update schematic
Parts:
- removed CN1: (no value), microbuilder:USB_TYPEAPTHFML
- added R28: R10K, resistor:R-EU_R0805
- added R29: R2K, resistor:R-EU_R0805
- added U$8: 74HC4053D, tigorcustom:74HC4053D
- V_SENSORS: device con-ptr500:AK300/4 -> con-ptr500:AK300/5
Connections:
- removed net N$17 (its old number): R16.1, V_SENSORS-4.KL
- new net N$19: R28.1, V_SENSORS-4.KL
- new net N$20: R16.1, V_SENSORS-5.KL
- new net N$34: R15.2
- new net SELECT_SENSOR: U$1.*10, U$8.S1
- new net SENSOR_HI_1: R14.2, R15.1, U$8.1Y1
- new net SENSOR_HI_2: R28.2, R29.1, U$8.1Y0
- net +3V3: no longer K1.1, K1.17
- net +5V: now also U$8.VCC; no longer CN1.VBUS
- net GND: now also R29.2, U$8./E, U$8.GND, U$8.VEE; no longer CN1.GND, R15.2
- net SENSOR_HUG_IDIR: now also U$8.1Z; no longer R14.2, R15.1
Other:
- moved on the sheet: R10, R11, R12, R13, R14, R15, R16, R17, V_SENSORS-1, V_SENSORS-2, V_SENSORS-3, V_SENSORS-4

Commit message: Update PCB design
Parts:
- removed B1: RECTIFIER-RB1A, rectifier:RECTIFIER-RB1A
- removed C2: C470uF, resistor:CPOL-EUE2-5
- removed D1: 5.1V, diode:ZENER-DIODEZD-7.5
- removed OK1: PC817, optocoupler:PC817
- removed R2: R470R, resistor:R-EU_0207/10
- removed R3: R270R, resistor:R-EU_M0805
- removed R4: R10K, resistor:R-EU_R0805
- added C14: C100N, resistor:C-EUC0805K
- added R30: R1K, resistor:R-EU_R0805
- added R31: R2K, resistor:R-EU_R0805
- added R32: R100K, resistor:R-EU_0309/V
- added R33: R2K, resistor:R-EU_0309/V
- added U$9: TRANSFORMER, bontor:TRANSFORMER
- R11: value R1K -> R2K
- R13: value R2K -> R1K
Connections:
- removed net N$17: R10.1, V_SENSORS-1.KL
- removed net N$34: R15.2
- removed net N$7: B1.+, C2.+, D1.C, OK1.A
- removed net N$8: B1.-, C2.-, D1.A, R3.1
- removed net N$9: OK1.C, R3.2
- new net N$35: R30.1, U$1.TXO
- new net N$36: R32.2, U$9.IA
- new net N$38: C14.2, R33.1, U$9.OB
- net +5V: no longer R4.1
- net AGND: now also C14.1
- net ARDU_TX: now also R30.2, R31.1; no longer U$1.TXO
- net CTRL_CHARGING: now also K1.11; no longer K1.12
- net CTRL_SIM_PWRKEY: now also K1.15
- net DHT_DATA: now also U$1.*10; no longer U$1.12
- net GND: now also R15.2, R31.2, V_ACCU-1.KL, V_LOAD-1.KL, V_PWR_SPLY-1.KL; no longer OK1.EMIT, V_ACCU-2.KL, V_LOAD-2.KL, V_PWR_SPLY-2.KL
- net N$1: now also R32.1, VAC-2.KL; no longer B1.AC1, VAC-1.KL
- net N$12: now also V_PWR_SPLY-2.KL; no longer V_PWR_SPLY-1.KL
- net N$2: now also U$9.IB, VAC-1.KL; no longer R2.1, VAC-2.KL
- net N$6: now also R12.1, V_SENSORS-2.KL; no longer B1.AC2, R2.2
- net SELECT_SENSOR: now also U$1.*6; no longer U$1.*10
- net SENSOR_BUC: now also R12.2, R13.1, U$1.A7; no longer R10.2, R11.1, U$1.A4
- net SENSOR_HUG_IDIR: now also U$1.A5; no longer U$1.A7
- net SENSOR_SCADA: now also U$1.A4; no longer U$1.A6
- net SENSOR_SCPC: now also R10.2, R11.1, U$1.A6; no longer R12.2, R13.1, U$1.A5
- net SENSOR_VAC: now also R33.2, U$9.OA; no longer OK1.COL, R4.2
- net USIM_DATA: now also D3.C1; no longer D3.C2
- net USIM_RST: now also D3.C2; no longer D3.C4
- net USIM_VDD: now also D3.C4; no longer D3.C1
- net VBAT: now also V_ACCU-2.KL; no longer V_ACCU-1.KL
- net VIN: now also R10.1, V_SENSORS-1.KL; no longer R12.1, V_SENSORS-2.KL
- net VLOAD: now also V_LOAD-2.KL; no longer V_LOAD-1.KL
Other:
- moved on the sheet: VAC-1, VAC-2, V_ACCU-1, V_ACCU-2, V_LOAD-1, V_LOAD-2, V_PWR_SPLY-1, V_PWR_SPLY-2
