File: board_sr/sr_indicator_v0/sr_indicator_v0.brd (EAGLE design)
At the start: 24 x 39 mm, 11 parts

Commit message: Finish routing
Parts:
- added IC1, IC2: ULN2004AD, uln-udn:SO16
- added LED11, LED12, LED13, LED14: (no value), adafruit:LED3MM
- added R1, R10, R11, R12, R13, R14, R2, R3, R4, R5, R6, R7, R8, R9: R220R, resistor:M0805
- CTRL_CONN: device con-lstb:MA06-2 -> con-lstb:MA08-2
- moved LED8 110.0 mm to (13.2, -89.8)
- moved LED9 109.6 mm to (2.75, -94.2)
- moved LED10 97.0 mm to (2.75, -80.8)
- moved CTRL_CONN 62.3 mm to (10.8, -54.0), flipped to the top
Connections:
- removed net +13.5V: CTRL_CONN.5, LED5.A
- removed net +19.5V: CTRL_CONN.6, LED6.A
- removed net +24V: CTRL_CONN.7, LED7.A
- removed net +6.5V: CTRL_CONN.4, LED4.A
- removed net VAC: CTRL_CONN.1, LED1.A
- removed net VBAT: CTRL_CONN.3, LED3.A
- removed net VBUC: CTRL_CONN.10, LED10.A
- removed net VPWR_SPLY: CTRL_CONN.2, LED2.A
- removed net VSCPC: CTRL_CONN.9, LED9.A
- removed net VWIFI: CTRL_CONN.8, LED8.A
- new net +5V: CTRL_CONN.15, LED1.A, LED10.A, LED11.A, LED12.A, LED13.A, LED14.A, LED2.A, LED3.A, LED4.A, LED5.A, LED6.A, LED7.A, LED8.A, LED9.A
- new net ARDU_FLASH: CTRL_CONN.1, IC1.1
- new net CTRL_LED0: CTRL_CONN.5, IC1.5
- new net CTRL_LED1: CTRL_CONN.6, IC1.6
- new net CTRL_LED2: CTRL_CONN.7, IC1.7
- new net CTRL_LED3: CTRL_CONN.8, IC2.1
- new net CTRL_LED4: CTRL_CONN.9, IC2.2
- new net CTRL_LED5: CTRL_CONN.10, IC2.3
- new net CTRL_LED6: CTRL_CONN.11, IC2.4
- new net CTRL_LED7: CTRL_CONN.12, IC2.5
- new net CTRL_LED8: CTRL_CONN.13, IC2.6
- new net CTRL_LED9: CTRL_CONN.14, IC2.7
- new net N$1: IC1.16, R1.1
- new net N$10: LED3.K, R3.2
- new net N$11: LED4.K, R4.2
- new net N$12: LED5.K, R5.2
- new net N$13: LED6.K, R6.2
- new net N$14: LED7.K, R7.2
- new net N$15: IC2.16, R8.1
- new net N$16: IC2.15, R9.1
- new net N$17: IC2.14, R10.1
- new net N$18: IC2.13, R11.1
- new net N$19: IC2.12, R12.1
- new net N$2: IC1.15, R2.1
- new net N$20: IC2.11, R13.1
- new net N$21: IC2.10, R14.1
- new net N$22: LED8.K, R8.2
- new net N$23: LED9.K, R9.2
- new net N$24: LED10.K, R10.2
- new net N$25: LED11.K, R11.2
- new net N$26: LED12.K, R12.2
- new net N$27: LED13.K, R13.2
- new net N$28: LED14.K, R14.2
- new net N$3: IC1.14, R3.1
- new net N$4: IC1.13, R4.1
- new net N$5: IC1.12, R5.1
- new net N$6: IC1.11, R6.1
- new net N$7: IC1.10, R7.1
- new net N$8: LED1.K, R1.2
- new net N$9: LED2.K, R2.2
- new net RPI_FLASH: CTRL_CONN.2, IC1.2
- new net SIM_NETLIGHT: CTRL_CONN.4, IC1.4
- new net SIM_STATUS: CTRL_CONN.3, IC1.3
- net GND: now also CTRL_CONN.16, IC1.8, IC2.8; no longer CTRL_CONN.11, CTRL_CONN.12, LED1.K, LED10.K, LED2.K, LED3.K, LED4.K, LED5.K, LED6.K, LED7.K, LED8.K, LED9.K
Routing:
- net GND: track 75.5 -> 0.00 mm
- net VAC: track 53.8 -> 0.00 mm
- net VBAT: track 44.4 -> 0.00 mm
- net +13.5V: track 35.0 -> 0.00 mm
- net VPWR_SPLY: track 30.9 -> 0.00 mm
- net +6.5V: track 26.6 -> 0.00 mm
- net +24V: track 25.5 -> 0.00 mm
- net +19.5V: track 22.5 -> 0.00 mm
- net VWIFI: track 18.5 -> 0.00 mm
- net VSCPC: track 16.1 -> 0.00 mm
- net VBUC: track 8.68 -> 0.00 mm
