File: board_sr/sr_controller_v1/sr_controller_v1.brd (EAGLE design)
At the start: 150 x 110 mm, 100 parts, among them Q1 32kHz, Q3 IRF5210

Commit message: Backup routing pcb
Parts:
- removed DUMMY_A, DUMMY_B, DUMMY_C, DUMMY_D: (no value), con-ptr500:AK300/2
- added F4: (no value), special:FUSE1
- added IC2, IC3: 74HC595D, 74xx-eu:SO16
- added INDICATOR: (no value), con-lstb:MA08-2
- added INDICATOR_OLD: (no value), con-lstb:MA06-2
- added R37, R40: R330R, resistor:R0805
- added R38, R39, R46: R2.7K, resistor:R0805
- added R41, R44: R1K, resistor:R0805
- added R42, R43, R45: R2K, resistor:R0805
- added R47: R10K, resistor:R0805
- R33: device resistor:0309V -> resistor:0309/10
- moved R3 64.6 mm to (38.0, 22.8), turned to 0 degrees
- moved X1 61.9 mm to (145.2, 41.5), turned to 270 degrees
- moved R29 61.4 mm to (38.0, 59.2), turned to 0 degrees
- moved R16 60.8 mm to (121.5, 96.0), turned to 270 degrees
- moved R15 60.3 mm to (38.0, 40.5), turned to 0 degrees
- moved R2 60.0 mm to (38.0, 25.2)
- moved R28 58.3 mm to (38.0, 61.8)
- moved R17 58.1 mm to (119.0, 96.0), turned to 90 degrees
- moved R14 55.9 mm to (38.0, 43.0)
- moved R10 42.2 mm to (97.5, 96.0), turned to 270 degrees
- moved R11 42.1 mm to (95.0, 96.0), turned to 90 degrees
- moved R34 40.9 mm to (57.0, 40.5), turned to 0 degrees
- moved U$8 40.7 mm to (66.0, 40.0), turned to 90 degrees
- moved R4 36.6 mm to (57.0, 43.0)
- moved BI_SPLY_A 36.5 mm to (9.00, 48.0)
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Connections:
- new net ARDU_FLASH: INDICATOR.1, U$1.12
- new net CTRL_LED0: IC2.15, INDICATOR.5
- new net CTRL_LED1: IC2.1, INDICATOR.6
- new net CTRL_LED2: IC2.2, INDICATOR.7
- new net CTRL_LED3: IC2.3, INDICATOR.8
- new net CTRL_LED4: IC2.4, INDICATOR.9
- new net CTRL_LED5: IC2.5, INDICATOR.10
- new net CTRL_LED6: IC2.6, INDICATOR.11
- new net CTRL_LED7: IC2.7, INDICATOR.12
- new net CTRL_LED8: IC3.15, INDICATOR.13
- new net CTRL_LED9: IC3.1, INDICATOR.14
- new net N$20: BI_SPLY_A.1, F4.1A
- new net N$34: INDICATOR_OLD.1, R37.2
- new net N$37: INDICATOR_OLD.2, R38.1
- new net N$39: INDICATOR_OLD.4, R40.1
- new net N$40: INDICATOR_OLD.5, R41.2
- new net N$41: INDICATOR_OLD.7, R43.2
- new net N$42: INDICATOR_OLD.9, R45.2
- new net N$43: INDICATOR_OLD.6, R42.1
- new net N$44: INDICATOR_OLD.8, R44.1
- new net N$45: INDICATOR_OLD.10, R46.1
- new net QS: IC2.9, IC3.14
- new net RPI_FLASH: INDICATOR.2, PCB1.13
- new net SR_DS: IC2.14, U$1.5
- new net SR_RST: IC2.10, IC3.10, R47.2, U$1.7
- new net SR_SHCP: IC2.11, IC3.11, U$1.6
- new net SR_STCP: IC2.12, IC3.12, U$1.8
- new net VPWR_SPLY: D2.C, Q3.S, R38.2, R5.1, V_PWR_SPLY.2
- net +13.5V: now also R39.1
- net +19.5V: now also R43.1
- net +5V: now also IC2.16, IC3.16, R47.1
- net +6.5V: now also R41.1
- net CTRL_CHARGING: now also PCB1.15; no longer PCB1.11
- net CTRL_SIM_PWRKEY: now also PCB1.11; no longer PCB1.15
- net GND: now also IC2.13, IC2.8, IC3.13, IC3.8, INDICATOR.15, INDICATOR.16, INDICATOR_OLD.11, INDICATOR_OLD.12; no longer PCB1.14, PCB1.20, PCB1.30, PCB1.34, PCB1.6
- net MDM_INDC_0: now also R35.2, U$1.16; no longer R36.2, U$1.15
- net MDM_INDC_1: now also R36.2, U$1.15; no longer R35.2, U$1.16
- net N$12: now also INDICATOR_OLD.3, R39.2; no longer D2.C, Q3.S, R5.1, V_PWR_SPLY.2
- net SEL_SENSOR_1: now also U$1.11; no longer U$1.9
- net SEL_SENSOR_3: now also U$1.9; no longer U$1.11
- net SENSOR_IBAT: now also U$1.17; no longer U$1.19
- net SENSOR_ILOAD: now also U$1.19; no longer U$1.20
- net SENSOR_MDM_1: now also U$8.5; no longer U$8.1
- net SENSOR_MDM_2: now also U$8.1; no longer U$8.5
- net SENSOR_VAC: now also R45.1, U$1.20; no longer U$1.17
- net SIM_NETLIGHT: now also INDICATOR.4
- net SIM_STATUS: now also INDICATOR.3
- net VBAT: now also R37.1
- net VLOAD: now also F4.2A, R44.2; no longer BI_SPLY_A.1
- net VMDM: now also R40.2
- net VSCADA: now also R46.2
- net VSCPC: now also R42.2
Routing:
- net GND: track 0.00 -> 348.8 mm, vias 0 -> 1
- net VMDM: track 0.00 -> 206.9 mm
- net VLOAD: track 0.00 -> 180.7 mm
- net VSCADA: track 0.00 -> 176.0 mm
- net VSCPC: track 0.00 -> 173.4 mm
- net SENSOR_VAC: track 0.00 -> 98.7 mm
- net VBAT: track 0.00 -> 60.0 mm, vias 0 -> 1
- net SENSOR_MDM_0: track 0.00 -> 59.8 mm
- net +13.5V: track 0.00 -> 55.7 mm
- net +6.5V: track 0.00 -> 48.8 mm
- net SENSOR_MDM_2: track 0.00 -> 44.8 mm
- net SENSOR_MDM_1: track 0.00 -> 42.6 mm, vias 0 -> 2
- net +5V: track 0.00 -> 39.6 mm
- net +19.5V: track 0.00 -> 36.2 mm
- net VPWR_SPLY: track 0.00 -> 30.7 mm
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
Commit message: Finish routing
Parts:
- removed IC3: 74HC595D, 74xx-eu:SO16
- removed INDICATOR: (no value), con-lstb:MA08-2
- removed INDICATOR_OLD: (no value), con-lstb:MA06-2
- removed U$3: GND_CONNECT, SparkFun-Passives:GND_CONNECT
- added INDICATOR_CONN: (no value), con-lstb:MA08-2
- added J2, J3, J4, J5, J6, J7: WIRE_HOLE-14AWG, powercube:WIRE_HOLE-14AWG
- added R48, R49, R50, R51: R10K, resistor:R0805
- added SJ3: (no value), microbuilder:SOLDERJUMPER_CLOSEDWIRE
- R23, R26: value R1K -> R220R
- R37, R40: value R330R -> R10K
- R38, R39, R46: value R2.7K -> R10K
- R41, R44: value R1K -> R10K
- R42, R43, R45: value R2K -> R10K
- moved IC2 152.4 mm to (127.8, 70.8), turned to 90 degrees
- moved R47 131.5 mm to (93.0, 66.0), flipped to the bottom, turned to 180 degrees
- moved R35 77.1 mm to (43.6, 14.0), turned to 180 degrees
- moved R36 76.7 mm to (43.6, 12.0), turned to 180 degrees
- moved R23 46.7 mm to (143.0, 49.5), turned to 270 degrees
- moved R27 44.4 mm to (130.5, 44.5), turned to 90 degrees
- moved T3 44.2 mm to (133.5, 44.5)
- moved R21 44.0 mm to (142.0, 40.2), turned to 180 degrees
- moved R22 41.1 mm to (142.0, 42.5), turned to 180 degrees
- moved T1 39.2 mm to (142.0, 45.5), turned to 0 degrees
- moved C8 39.0 mm to (145.8, 19.5), turned to 90 degrees
- moved U$5 35.0 mm to (140.5, 18.0)
- moved R18 34.1 mm to (103.0, 2.75)
- moved R19 34.1 mm to (100.5, 2.75)
- moved C10 34.1 mm to (97.2, 12.0)
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Connections:
- removed net N$12: INDICATOR_OLD.3, R39.2
- removed net N$15: Q3.D, U$4.1, U$4.2
- removed net N$34: INDICATOR_OLD.1, R37.2
- removed net N$37: INDICATOR_OLD.2, R38.1
- removed net N$39: INDICATOR_OLD.4, R40.1
- removed net N$40: INDICATOR_OLD.5, R41.2
- removed net N$41: INDICATOR_OLD.7, R43.2
- removed net N$42: INDICATOR_OLD.9, R45.2
- removed net N$43: INDICATOR_OLD.6, R42.1
- removed net N$44: INDICATOR_OLD.8, R44.1
- removed net N$45: INDICATOR_OLD.10, R46.1
- removed net QS: IC2.9, IC3.14
- new net RPI_3V3: PCB1.17, R35.1, R36.1
- new net VSPLY: Q3.D, U$2.1, U$2.2, U$4.1, U$4.2
- net +13.5V: no longer R39.1
- net +19.5V: no longer R43.1
- net +3V3: now also R37.1, R38.1, R44.1
- net +5V: now also INDICATOR_CONN.15, R39.1, R40.1, R41.1, R42.1, R43.1, R45.1, R46.1, R48.1, R49.1, R50.1, R51.1; no longer IC3.16, R35.1, R36.1
- net +6.5V: no longer R41.1
- net AGND: now also SJ3.2; no longer U$3.2
- net ARDU_FLASH: now also INDICATOR_CONN.4, R45.2, U$1.14; no longer INDICATOR.1, U$1.12
- net ARDU_RX: now also PCB1.31; no longer PCB1.35
- net ARDU_TX: now also PCB1.33; no longer PCB1.37
- net CTRL_CHARGING: now also PCB1.40; no longer PCB1.15
- net CTRL_LED0: now also INDICATOR_CONN.13, R43.2; no longer INDICATOR.5
- net CTRL_LED1: now also INDICATOR_CONN.14, R51.2; no longer INDICATOR.6
- net CTRL_LED2: now also INDICATOR_CONN.11, R42.2; no longer INDICATOR.7
- net CTRL_LED3: now also INDICATOR_CONN.12, R50.2; no longer INDICATOR.8
- net CTRL_LED4: now also INDICATOR_CONN.9, R41.2; no longer INDICATOR.9
- net CTRL_LED5: now also INDICATOR_CONN.10, R49.2; no longer INDICATOR.10
- net CTRL_LED6: now also INDICATOR_CONN.7, R40.2; no longer INDICATOR.11
- net CTRL_LED7: now also INDICATOR_CONN.8, R48.2; no longer INDICATOR.12
- net CTRL_LED8: now also INDICATOR_CONN.5, R39.2, U$1.15; no longer IC3.15, INDICATOR.13
- net CTRL_LED9: now also INDICATOR_CONN.6, R46.2, U$1.16; no longer IC3.1, INDICATOR.14
- net GND: now also INDICATOR_CONN.16, SJ3.1; no longer IC3.13, IC3.8, INDICATOR.15, INDICATOR.16, INDICATOR_OLD.11, INDICATOR_OLD.12, U$3.1
- net MDM_INDC_0: now also PCB1.35, R36.2; no longer R35.2, U$1.16
- net MDM_INDC_1: now also PCB1.37, R35.2; no longer R36.2, U$1.15
- net RPI_FLASH: now also INDICATOR_CONN.3, R38.2; no longer INDICATOR.2
- net SENSOR_IBAT: now also U$1.20; no longer U$1.17
- net SENSOR_ILOAD: now also U$1.18; no longer U$1.19
- net SENSOR_SCADA: now also U$1.27; no longer U$1.25
- net SENSOR_SCPC: now also U$1.25; no longer U$1.27
- net SENSOR_VAC: now also U$1.17; no longer R45.1, U$1.20
- net SENSOR_VBAT: now also U$1.19; no longer U$1.18
- net SIM_NETLIGHT: now also INDICATOR_CONN.1, R37.2; no longer INDICATOR.4
- net SIM_STATUS: now also INDICATOR_CONN.2, R44.2; no longer INDICATOR.3
- net SR_DS: now also U$1.8; no longer U$1.5
- net SR_RST: now also U$1.5; no longer IC3.10, U$1.7
- net SR_SHCP: no longer IC3.11
- net SR_STCP: now also U$1.7; no longer IC3.12, U$1.8
- net VBAT: no longer R37.1, U$2.1, U$2.2
- net VLOAD: now also J2.P$1, J3.P$1; no longer R44.2
- net VMDM: no longer R40.2
- net VPWR_SPLY: no longer R38.2
- net VSCADA: now also J6.P$1, J7.P$1; no longer R46.2
- net VSCPC: now also J4.P$1, J5.P$1; no longer R42.2
Routing:
- net GND: track 348.8 -> 978.3 mm, vias 1 -> 15
- net +5V: track 39.6 -> 504.0 mm, vias 0 -> 16
- net SENSOR_VBAT: track 2.30 -> 175.0 mm, vias 0 -> 1
- net SENSOR_ILOAD: track 0.00 -> 169.1 mm
- net SENSOR_IBAT: track 0.00 -> 167.2 mm, vias 0 -> 2
- net +3V3: track 0.00 -> 149.5 mm, vias 0 -> 3
- net CTRL_CHARGING: track 0.00 -> 136.8 mm, vias 0 -> 1
- net RPI_FLASH: track 0.00 -> 122.5 mm, vias 0 -> 5
- net ARDU_TX: track 0.00 -> 114.8 mm, vias 0 -> 1
- net ARDU_RX: track 0.00 -> 112.2 mm, vias 0 -> 2
- net VMDM: track 206.9 -> 143.3 mm
- net SIM_NETLIGHT: track 0.00 -> 57.9 mm, vias 0 -> 2
- net CTRL_SIM_PWRKEY: track 28.5 -> 85.3 mm, vias 0 -> 2
- net CTRL_LED0: track 0.00 -> 55.3 mm
- net SENSOR_VAC: track 98.7 -> 153.4 mm
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- added copper zone on layer 1, net GND
- added copper zone on layer 16, net GND
- added copper zone on layer 16, net N$12

Commit message: Finish Routing PCB ver1 revA
Parts:
- removed D2: 18V, diode:DO41Z10
- removed Q3: IRF5210, transistor-power:TO220BV
- removed R5: R10K, resistor:R0805
- removed R9: R20K, resistor:R0805
- added D1: 1N4007, diode:DO214AA
- added K1: G5L, relay:G5LE
Connections:
- removed net N$11: D2.A, Q3.G, R5.2, R9.1
- removed net N$14: R9.2, T4.C
- new net N$34: D1.A, K1.2, T4.C
- net VPWR_SPLY: now also K1.P; no longer D2.C, Q3.S, R5.1
- net VSCADA: now also D1.C, K1.1
- net VSPLY: now also K1.S; no longer Q3.D
Routing:
- net N$11: track 24.9 -> 0.00 mm
- net VPWR_SPLY: track 30.7 -> 10.4 mm
- net VSPLY: track 14.4 -> 0.00 mm
- net RPI_FLASH: track 122.5 -> 132.8 mm
- net N$14: track 2.85 -> 0.00 mm
- net SENSOR_MDM_2: track 44.4 -> 43.2 mm
- net ARDU_RX: track 112.2 -> 111.5 mm
- net ARDU_TX: track 114.8 -> 114.2 mm
- net SENSOR_MDM_0: track 60.0 -> 59.4 mm
