File: board_sr/sr_controller_v1/sr_controller_v1.sch (EAGLE design)
At the start: 100 parts, among them Q1 32kHz, Q3 IRF5210

Commit message: Backup routing pcb
Parts:
- removed DUMMY_A, DUMMY_B, DUMMY_C, DUMMY_D: (no value), con-ptr500:AK300/2
- added F4: (no value), special:FUSE2P
- added IC2, IC3: 74HC595D, 74xx-eu:74HC595D
- added INDICATOR: (no value), con-lstb:MA08-2
- added INDICATOR_OLD: (no value), con-lstb:MA06-2
- added R37, R40: R330R, resistor:R-EU_R0805
- added R38, R39, R46: R2.7K, resistor:R-EU_R0805
- added R41, R44: R1K, resistor:R-EU_R0805
- added R42, R43, R45: R2K, resistor:R-EU_R0805
- added R47: R10K, resistor:R-EU_R0805
- R33: device resistor:R-EU_0309/V -> resistor:R-EU_0309/10
Connections:
- new net ARDU_FLASH: INDICATOR.1, U$1.*9
- new net CTRL_LED0: IC2A.QA, INDICATOR.5
- new net CTRL_LED1: IC2A.QB, INDICATOR.6
- new net CTRL_LED2: IC2A.QC, INDICATOR.7
- new net CTRL_LED3: IC2A.QD, INDICATOR.8
- new net CTRL_LED4: IC2A.QE, INDICATOR.9
- new net CTRL_LED5: IC2A.QF, INDICATOR.10
- new net CTRL_LED6: IC2A.QG, INDICATOR.11
- new net CTRL_LED7: IC2A.QH, INDICATOR.12
- new net CTRL_LED8: IC3A.QA, INDICATOR.13
- new net CTRL_LED9: IC3A.QB, INDICATOR.14
- new net N$20: BI_SPLY_A-1.KL, F4.1A
- new net N$34: INDICATOR_OLD.1, R37.2
- new net N$37: INDICATOR_OLD.2, R38.1
- new net N$39: INDICATOR_OLD.4, R40.1
- new net N$40: INDICATOR_OLD.5, R41.2
- new net N$41: INDICATOR_OLD.7, R43.2
- new net N$42: INDICATOR_OLD.9, R45.2
- new net N$43: INDICATOR_OLD.6, R42.1
- new net N$44: INDICATOR_OLD.8, R44.1
- new net N$45: INDICATOR_OLD.10, R46.1
- new net QS: IC2A.QH*, IC3A.SER
- new net RPI_FLASH: INDICATOR.2, PCB1.GPIO27/GEN2
- new net SR_DS: IC2A.SER, U$1.2
- new net SR_RST: IC2A.SCL, IC3A.SCL, R47.2, U$1.4
- new net SR_SHCP: IC2A.SCK, IC3A.SCK, U$1.*3
- new net SR_STCP: IC2A.RCK, IC3A.RCK, U$1.*5
- new net VPWR_SPLY: D2.C, Q3.S, R38.2, R5.1, V_PWR_SPLY-2.KL
- net +13.5V: now also R39.1
- net +19.5V: now also R43.1
- net +5V: now also IC2P.VCC, IC3P.VCC, R47.1
- net +6.5V: now also R41.1
- net CTRL_CHARGING: now also PCB1.GPIO22/GEN3; no longer PCB1.GPIO17/GEN0
- net CTRL_SIM_PWRKEY: now also PCB1.GPIO17/GEN0; no longer PCB1.GPIO22/GEN3
- net GND: now also IC2A.G, IC2P.GND, IC3A.G, IC3P.GND, INDICATOR.15, INDICATOR.16, INDICATOR_OLD.11, INDICATOR_OLD.12; no longer PCB1.GND@4, PCB1.GND@5, PCB1.GND@6, PCB1.GND@7, PCB1.GND@8
- net MDM_INDC_0: now also R35.2, U$1.13; no longer R36.2, U$1.12
- net MDM_INDC_1: now also R36.2, U$1.12; no longer R35.2, U$1.13
- net N$12: now also INDICATOR_OLD.3, R39.2; no longer D2.C, Q3.S, R5.1, V_PWR_SPLY-2.KL
- net SEL_SENSOR_1: now also U$1.8; no longer U$1.*6
- net SEL_SENSOR_3: now also U$1.*6; no longer U$1.8
- net SENSOR_IBAT: now also U$1.A0; no longer U$1.A2
- net SENSOR_ILOAD: now also U$1.A2; no longer U$1.A3
- net SENSOR_MDM_1: now also U$8.3Y0; no longer U$8.2Y1
- net SENSOR_MDM_2: now also U$8.2Y1; no longer U$8.3Y0
- net SENSOR_VAC: now also R45.1, U$1.A3; no longer U$1.A0
- net SIM_NETLIGHT: now also INDICATOR.4
- net SIM_STATUS: now also INDICATOR.3
- net VBAT: now also R37.1
- net VLOAD: now also F4.2A, R44.2; no longer BI_SPLY_A-1.KL
- net VMDM: now also R40.2
- net VSCADA: now also R46.2
- net VSCPC: now also R42.2
Other:
- moved on the sheet: BI_REG_A-1, BI_REG_A-2, BI_REG_B-1, BI_REG_B-2, F1, F2, F3, MDM_REG_A-1, MDM_REG_A-2, MDM_REG_B-1, MDM_REG_B-2, SCADA_REG_A-1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

Commit message: Finish routing
Parts:
- removed IC3: 74HC595D, 74xx-eu:74HC595D
- removed INDICATOR: (no value), con-lstb:MA08-2
- removed INDICATOR_OLD: (no value), con-lstb:MA06-2
- removed U$3: GND_CONNECT, SparkFun-Passives:GND_CONNECT
- added INDICATOR_CONN: (no value), con-lstb:MA08-2
- added J2, J3, J4, J5, J6, J7: WIRE_HOLE-14AWG, powercube:WIRE_HOLE-14AWG
- added R48, R49, R50, R51: R10K, resistor:R-EU_R0805
- added SJ3: (no value), microbuilder:SOLDERJUMPERCLOSED
- R23, R26: value R1K -> R220R
- R37, R40: value R330R -> R10K
- R38, R39, R46: value R2.7K -> R10K
- R41, R44: value R1K -> R10K
- R42, R43, R45: value R2K -> R10K
Connections:
- removed net N$12: INDICATOR_OLD.3, R39.2
- removed net N$15: Q3.D, U$4.IP+@1, U$4.IP+@2
- removed net N$34: INDICATOR_OLD.1, R37.2
- removed net N$37: INDICATOR_OLD.2, R38.1
- removed net N$39: INDICATOR_OLD.4, R40.1
- removed net N$40: INDICATOR_OLD.5, R41.2
- removed net N$41: INDICATOR_OLD.7, R43.2
- removed net N$42: INDICATOR_OLD.9, R45.2
- removed net N$43: INDICATOR_OLD.6, R42.1
- removed net N$44: INDICATOR_OLD.8, R44.1
- removed net N$45: INDICATOR_OLD.10, R46.1
- removed net QS: IC2A.QH*, IC3A.SER
- new net RPI_3V3: PCB1.3V3@2, R35.1, R36.1
- new net VSPLY: Q3.D, U$2.IP+@1, U$2.IP+@2, U$4.IP+@1, U$4.IP+@2
- net +13.5V: no longer R39.1
- net +19.5V: no longer R43.1
- net +3V3: now also R37.1, R38.1, R44.1
- net +5V: now also INDICATOR_CONN.15, R39.1, R40.1, R41.1, R42.1, R43.1, R45.1, R46.1, R48.1, R49.1, R50.1, R51.1; no longer IC3P.VCC, R35.1, R36.1
- net +6.5V: no longer R41.1
- net AGND: now also SJ3.2; no longer U$3.AGND
- net ARDU_FLASH: now also INDICATOR_CONN.4, R45.2, U$1.*11; no longer INDICATOR.1, U$1.*9
- net ARDU_RX: now also PCB1.GPIO6; no longer PCB1.GPIO19
- net ARDU_TX: now also PCB1.GPIO13; no longer PCB1.GPIO26
- net CTRL_CHARGING: now also PCB1.GPIO21; no longer PCB1.GPIO22/GEN3
- net CTRL_LED0: now also INDICATOR_CONN.13, R43.2; no longer INDICATOR.5
- net CTRL_LED1: now also INDICATOR_CONN.14, R51.2; no longer INDICATOR.6
- net CTRL_LED2: now also INDICATOR_CONN.11, R42.2; no longer INDICATOR.7
- net CTRL_LED3: now also INDICATOR_CONN.12, R50.2; no longer INDICATOR.8
- net CTRL_LED4: now also INDICATOR_CONN.9, R41.2; no longer INDICATOR.9
- net CTRL_LED5: now also INDICATOR_CONN.10, R49.2; no longer INDICATOR.10
- net CTRL_LED6: now also INDICATOR_CONN.7, R40.2; no longer INDICATOR.11
- net CTRL_LED7: now also INDICATOR_CONN.8, R48.2; no longer INDICATOR.12
- net CTRL_LED8: now also INDICATOR_CONN.5, R39.2, U$1.12; no longer IC3A.QA, INDICATOR.13
- net CTRL_LED9: now also INDICATOR_CONN.6, R46.2, U$1.13; no longer IC3A.QB, INDICATOR.14
- net GND: now also INDICATOR_CONN.16, SJ3.1; no longer IC3A.G, IC3P.GND, INDICATOR.15, INDICATOR.16, INDICATOR_OLD.11, INDICATOR_OLD.12, U$3.DGND
- net MDM_INDC_0: now also PCB1.GPIO19, R36.2; no longer R35.2, U$1.13
- net MDM_INDC_1: now also PCB1.GPIO26, R35.2; no longer R36.2, U$1.12
- net RPI_FLASH: now also INDICATOR_CONN.3, R38.2; no longer INDICATOR.2
- net SENSOR_IBAT: now also U$1.A3; no longer U$1.A0
- net SENSOR_ILOAD: now also U$1.A1; no longer U$1.A2
- net SENSOR_SCADA: now also U$1.A6; no longer U$1.A4
- net SENSOR_SCPC: now also U$1.A4; no longer U$1.A6
- net SENSOR_VAC: now also U$1.A0; no longer R45.1, U$1.A3
- net SENSOR_VBAT: now also U$1.A2; no longer U$1.A1
- net SIM_NETLIGHT: now also INDICATOR_CONN.1, R37.2; no longer INDICATOR.4
- net SIM_STATUS: now also INDICATOR_CONN.2, R44.2; no longer INDICATOR.3
- net SR_DS: now also U$1.*5; no longer U$1.2
- net SR_RST: now also U$1.2; no longer IC3A.SCL, U$1.4
- net SR_SHCP: no longer IC3A.SCK
- net SR_STCP: now also U$1.4; no longer IC3A.RCK, U$1.*5
- net VBAT: no longer R37.1, U$2.IP+@1, U$2.IP+@2
- net VLOAD: now also J2.P$1, J3.P$1; no longer R44.2
- net VMDM: no longer R40.2
- net VPWR_SPLY: no longer R38.2
- net VSCADA: now also J6.P$1, J7.P$1; no longer R46.2
- net VSCPC: now also J4.P$1, J5.P$1; no longer R42.2
Other:
- moved on the sheet: IC2, IC2P, R35, R36, R37, R38, R39, R40, R41, R42, R43, R44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

Commit message: Finish Routing PCB ver1 revA
Parts:
- removed D2: 18V, diode:ZENER-DIODEDO41Z10
- removed Q3: IRF5210, transistor-power:PMOSFET_PTO220BV
- removed R5: R10K, resistor:R-EU_R0805
- removed R9: R20K, resistor:R-EU_R0805
- added D1: 1N4007, diode:DIODE-DO214AA
- added K1: G5L, relay:G5L
Connections:
- removed net N$11: D2.A, Q3.G, R5.2, R9.1
- removed net N$14: R9.2, T4.C
- new net N$34: D1.A, K11.2, T4.C
- net VPWR_SPLY: now also K12.P; no longer D2.C, Q3.S, R5.1
- net VSCADA: now also D1.C, K11.1
- net VSPLY: now also K12.S; no longer Q3.D
Other:
- moved on the sheet: R6, T4, V_PWR_SPLY-1, V_PWR_SPLY-2
Changed lines of the file:
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@@
 <part name="V_PWR_SPLY" library="con-ptr500" deviceset="AK300/2" device=""/>
 <part name="V_ACCU" library="con-ptr500" deviceset="AK300/2" device=""/>
-<part name="Q3" library="transistor-power" deviceset="PMOSFET_P" device="TO220BV" value="IRF5210"/>
 <part name="GND15" library="supply1" deviceset="GND" device=""/>
-<part name="R5" library="resistor" deviceset="R-EU_" device="R0805" value="R10K"/>
 <part name="GND16" library="supply1" deviceset="GND" device=""/>
 <part name="GND17" library="supply1" deviceset="GND" device=""/>
@@
 <part name="AGND3" library="supply1" deviceset="AGND" device=""/>
 <part name="GND19" library="supply1" deviceset="GND" device=""/>
-<part name="R9" library="resistor" deviceset="R-EU_" device="R0805" value="R20K"/>
-<part name="D2" library="diode" deviceset="ZENER-DIODE" device="DO41Z10" value="18V"/>
 <part name="U$4" library="SparkFun-AnalogIC" deviceset="ACS712" device=""/>
 <part name="C5" library="resistor" deviceset="C-EU" device="C0805K" value="C100N"/>
@@
 <part name="J6" library="powercube" deviceset="WIRE_HOLE-14AWG" device=""/>
 <part name="J7" library="powercube" deviceset="WIRE_HOLE-14AWG" device=""/>
+<part name="K1" library="relay" deviceset="G5L" device=""/>
+<part name="D1" library="diode" deviceset="DIODE-" device="DO214AA" value="1N4007"/>
 </parts>
 <sheets>
@@
 <instance part="VAC" gate="-1" x="177.8" y="231.14"/>
 <instance part="VAC" gate="-2" x="177.8" y="236.22"/>
-<instance part="V_PWR_SPLY" gate="-1" x="231.14" y="185.42"/>
-<instance part="V_PWR_SPLY" gate="-2" x="231.14" y="190.5"/>
+<instance part="V_PWR_SPLY" gate="-1" x="238.76" y="193.04"/>
+<instance part="V_PWR_SPLY" gate="-2" x="238.76" y="198.12"/>
 <instance part="V_ACCU" gate="-1" x="269.24" y="142.24" rot="R180"/>
 <instance part="V_ACCU" gate="-2" x="269.24" y="147.32" rot="R180"/>
-<instance part="Q3" gate="G$1" x="261.62" y="172.72"/>
 <instance part="GND15" gate="1" x="264.16" y="137.16"/>
-<instance part="R5" gate="G$1" x="243.84" y="182.88" rot="R270"/>
-<instance part="GND16" gate="1" x="236.22" y="180.34"/>
-<instance part="GND17" gate="1" x="243.84" y="137.16"/>
-<instance part="R6" gate="G$1" x="231.14" y="154.94"/>
+<instance part="GND16" gate="1" x="243.84" y="187.96"/>
+<instance part="GND17" gate="1" x="228.6" y="144.78"/>
+<instance part="R6" gate="G$1" x="215.9" y="154.94"/>
 <instance part="R7" gate="G$1" x="287.02" y="223.52" rot="R270"/>
 <instance part="R8" gate="G$1" x="287.02" y="210.82" rot="R270"/>
@@
 <instance part="AGND3" gate="VR1" x="320.04" y="213.36"/>
 <instance part="GND19" gate="1" x="309.88" y="213.36"/>
-<instance part="R9" gate="G$1" x="243.84" y="167.64" rot="R270"/>
-<instance part="D2" gate="G$1" x="251.46" y="182.88" rot="R90"/>
 <instance part="U$4" gate="G$1" x="279.4" y="157.48"/>
 <instance part="C5" gate="G$1" x="299.72" y="170.18" rot="R180"/>
@@
 <instance part="U$6" gate="G$1" x="48.26" y="78.74"/>
 <instance part="U$7" gate="G$1" x="48.26" y="45.72"/>
-<instance part="T4" gate="G$1" x="241.3" y="154.94"/>
+<instance part="T4" gate="G$1" x="226.06" y="154.94"/>
 <instance part="U$8" gate="G$1" x="347.98" y="106.68"/>
 <instance part="GND45" gate="1" x="335.28" y="93.98"/>
@@
 <instance part="J6" gate="G$1" x="398.78" y="160.02"/>
 <instance part="J7" gate="G$1" x="398.78" y="149.86"/>
+<instance part="K1" gate="1" x="228.6" y="167.64"/>
+<instance part="K1" gate="2" x="246.38" y="167.64"/>
+<instance part="D1" gate="G$1" x="236.22" y="167.64" rot="R90"/>
 </instances>
 <busses>
@@
 </segment>
 <segment>
-<wire x1="243.84" y1="149.86" x2="243.84" y2="139.7" width="0.1524" layer="91"/>
+<wire x1="228.6" y1="149.86" x2="228.6" y2="147.32" width="0.1524" layer="91"/>
 <pinref part="GND17" gate="1" pin="GND"/>
 <pinref part="T4" gate="G$1" pin="E"/>
@@
 <pinref part="GND16" gate="1" pin="GND"/>
 <pinref part="V_PWR_SPLY" gate="-1" pin="KL"/>
-<wire x1="236.22" y1="182.88" x2="236.22" y2="185.42" width="0.1524" layer="91"/>
+<wire x1="243.84" y1="190.5" x2="243.84" y2="193.04" width="0.1524" layer="91"/>
 </segment>
 <segment>
@@
 </segment>
 </net>
-<net name="N$11" class="0">
-<segment>
-<pinref part="Q3" gate="G$1" pin="G"/>
-<pinref part="R5" gate="G$1" pin="2"/>
-<wire x1="243.84" y1="177.8" x2="243.84" y2="175.26" width="0.1524" layer="91"/>
-<wire x1="256.54" y1="175.26" x2="251.46" y2="175.26" width="0.1524" layer="91"/>
-<pinref part="D2" gate="G$1" pin="A"/>
-<wire x1="251.46" y1="175.26" x2="243.84" y2="175.26" width="0.1524" layer="91"/>
-<wire x1="251.46" y1="180.34" x2="251.46" y2="175.26" width="0.1524" layer="91"/>
-<pinref part="R9" gate="G$1" pin="1"/>
-<wire x1="243.84" y1="172.72" x2="243.84" y2="175.26" width="0.1524" layer="91"/>
-</segment>
-</net>
 <net name="VPWR_SPLY" class="0">
 <segment>
-<pinref part="Q3" gate="G$1" pin="S"/>
-<wire x1="243.84" y1="190.5" x2="251.46" y2="190.5" width="0.1524" layer="91"/>
-<wire x1="251.46" y1="190.5" x2="264.16" y2="190.5" width="0.1524" layer="91"/>
-<wire x1="264.16" y1="190.5" x2="264.16" y2="180.34" width="0.1524" layer="91"/>
-<pinref part="R5" gate="G$1" pin="1"/>
-<wire x1="264.16" y1="180.34" x2="264.16" y2="177.8" width="0.1524" layer="91"/>
-<wire x1="243.84" y1="187.96" x2="243.84" y2="190.5" width="0.1524" layer="91"/>
-<pinref part="D2" gate="G$1" pin="C"/>
-<wire x1="251.46" y1="185.42" x2="251.46" y2="190.5" width="0.1524" layer="91"/>
 <pinref part="V_PWR_SPLY" gate="-2" pin="KL"/>
-<wire x1="236.22" y1="190.5" x2="243.84" y2="190.5" width="0.1524" layer="91"/>
-<label x="266.7" y="180.34" size="0.8128" layer="95" xref="yes"/>
-<wire x1="266.7" y1="180.34" x2="264.16" y2="180.34" width="0.1524" layer="91"/>
+<wire x1="243.84" y1="198.12" x2="246.38" y2="198.12" width="0.1524" layer="91"/>
+<label x="246.38" y="198.12" size="0.8128" layer="95" xref="yes"/>
+</segment>
+<segment>
+<pinref part="K1" gate="2" pin="P"/>
+<wire x1="246.38" y1="165.1" x2="246.38" y2="162.56" width="0.1524" layer="91"/>
+<label x="246.38" y="162.56" size="0.8128" layer="95" rot="R270" xref="yes"/>
 </segment>
 </net>
@@
 <segment>
 <pinref part="R6" gate="G$1" pin="2"/>
-<wire x1="238.76" y1="154.94" x2="236.22" y2="154.94" width="0.1524" layer="91"/>
+<wire x1="223.52" y1="154.94" x2="220.98" y2="154.94" width="0.1524" layer="91"/>
 <pinref part="T4" gate="G$1" pin="B"/>
 </segment>
@@
 <segment>
 <pinref part="R6" gate="G$1" pin="1"/>
-<wire x1="226.06" y1="154.94" x2="223.52" y2="154.94" width="0.1524" layer="91"/>
-<label x="223.52" y="154.94" size="0.8128" layer="95" rot="R180" xref="yes"/>
+<wire x1="210.82" y1="154.94" x2="208.28" y2="154.94" width="0.1524" layer="91"/>
+<label x="208.28" y="154.94" size="0.8128" layer="95" rot="R180" xref="yes"/>
 </segment>
 <segment>
@@
 </segment>
 </net>
-<net name="N$14" class="0">
-<segment>
-<pinref part="R9" gate="G$1" pin="2"/>
-<wire x1="243.84" y1="160.02" x2="243.84" y2="162.56" width="0.1524" layer="91"/>
-<pinref part="T4" gate="G$1" pin="C"/>
-</segment>
-</net>
 <net name="VSPLY" class="0">
 <segment>
-<pinref part="Q3" gate="G$1" pin="D"/>
 <pinref part="U$4" gate="G$1" pin="IP+@1"/>
-<wire x1="264.16" y1="167.64" x2="264.16" y2="162.56" width="0.1524" layer="91"/>
 <pinref part="U$4" gate="G$1" pin="IP+@2"/>
 <wire x1="264.16" y1="162.56" x2="264.16" y2="160.02" width="0.1524" layer="91"/>
@@
 <wire x1="332.74" y1="228.6" x2="330.2" y2="228.6" width="0.1524" layer="91"/>
 <label x="330.2" y="228.6" size="0.8128" layer="95" rot="R180" xref="yes"/>
+</segment>
+<segment>
+<pinref part="K1" gate="2" pin="S"/>
+<wire x1="241.3" y1="172.72" x2="241.3" y2="175.26" width="0.1524" layer="91"/>
+<label x="241.3" y="175.26" size="0.8128" layer="95" rot="R90" xref="yes"/>
 </segment>
 </net>
@@
 <label x="403.86" y="149.86" size="0.8128" layer="95" xref="yes"/>
 </segment>
+<segment>
+<pinref part="K1" gate="1" pin="1"/>
+<pinref part="D1" gate="G$1" pin="C"/>
+<wire x1="228.6" y1="172.72" x2="236.22" y2="172.72" width="0.1524" layer="91"/>
+<wire x1="236.22" y1="172.72" x2="236.22" y2="170.18" width="0.1524" layer="91"/>
+<wire x1="228.6" y1="172.72" x2="226.06" y2="172.72" width="0.1524" layer="91"/>
+<label x="226.06" y="172.72" size="0.8128" layer="95" rot="R180" xref="yes"/>
+</segment>
 </net>
 <net name="VSCPC" class="0">
@@
 </segment>
 </net>
+<net name="N$34" class="0">
+<segment>
+<pinref part="K1" gate="1" pin="2"/>
+<pinref part="D1" gate="G$1" pin="A"/>
+<wire x1="228.6" y1="162.56" x2="236.22" y2="162.56" width="0.1524" layer="91"/>
+<wire x1="236.22" y1="162.56" x2="236.22" y2="165.1" width="0.1524" layer="91"/>
+<pinref part="T4" gate="G$1" pin="C"/>
+<wire x1="228.6" y1="162.56" x2="228.6" y2="160.02" width="0.1524" layer="91"/>
+</segment>
+</net>
