File: board_sr/sr_controller_v1/sr_controller_v1_revB.brd (EAGLE design)
At the start: 140 x 150 mm, 126 parts, among them IC2 74HC595D, J2 WIRE_HOLE-14AWG, J3 WIRE_HOLE-14AWG, J4 WIRE_HOLE-14AWG, J5 WIRE_HOLE-14AWG, J6 WIRE_HOLE-14AWG, J7 WIRE_HOLE-14AWG, J8 WIRE_HOLE-14AWG, J9 WIRE_HOLE-14AWG, K1 G5L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

Commit message: Publish sr_controller_v1_revC
Other:
- board text added: "J2"
- board text added: "J3"
- board text added: "J4"
- board text added: "J5"
- board text added: "J6"
- board text added: "J7"
- board text added: "J8"
- board text added: "J9"
Changed lines of the file:
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@@
 <wire x1="18.5" y1="22" x2="20" y2="20.5" width="0" layer="20" curve="-90"/>
 <wire x1="21.5" y1="0" x2="20" y2="1.5" width="0" layer="20" curve="-90"/>
+<text x="26" y="109.75" size="1.778" layer="25">J5</text>
+<text x="46.25" y="108" size="1.778" layer="25">J4</text>
+<text x="40.25" y="99" size="1.778" layer="25">J3</text>
+<text x="42" y="58" size="1.778" layer="25">J2</text>
+<text x="19" y="34.75" size="1.778" layer="25">J6</text>
+<text x="26.75" y="22.75" size="1.778" layer="25">J7</text>
+<text x="27" y="12.75" size="1.778" layer="25">J8</text>
+<text x="45.5" y="33.25" size="1.778" layer="25">J9</text>
 </plain>
 <attributes>
