File: board_sr/sr_controller_v1/sr_controller_v1_revC.brd (EAGLE design)
At the start: 130 x 150 mm, 96 parts, among them IC3 LM741D, J2 WIRE_HOLE-14AWG, J3 WIRE_HOLE-14AWG, J4 WIRE_HOLE-14AWG, J5 WIRE_HOLE-14AWG, J6 WIRE_HOLE-14AWG, J7 WIRE_HOLE-14AWG, J8 WIRE_HOLE-14AWG, J9 WIRE_HOLE-14AWG, Q1 32kHz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

Commit message: Update sr_controller_v1_revC
Parts:
- removed FROM_LTC_REG: (no value), con-ptr500:AK300/2
- added FROM_LTC_REG_A, FROM_LTC_REG_B: (no value), con-ptr500:AK300/2
- C6: value C1NF -> C1nF
- R33: value R5K1 -> R5.1K
- moved T1 6.09 mm to (44.8, 14.0), turned to 90 degrees
- moved R20 5.94 mm to (49.2, 15.0)
- moved R21 5.94 mm to (49.2, 13.0)
- moved D1 5.22 mm to (41.5, 9.75), turned to 90 degrees
- moved FROM_GREY_REG 3.00 mm to (76.0, 18.0)
- moved TO_GREY_REG 3.00 mm to (86.0, 18.0)
- moved TO_LTC_REG 3.00 mm to (101.0, 18.0)
- flipped BAT1 to the top
- flipped Q1 to the top
Connections:
- net +12V: now also FROM_LTC_REG_B.1; no longer FROM_LTC_REG.2
- net +13V5: now also FROM_LTC_REG_A.2
- net +19V5: now also FROM_LTC_REG_A.1; no longer FROM_LTC_REG.1
- net +6V5: now also FROM_LTC_REG_B.2
- net N$3: now also Q1.2; no longer Q1.1
- net N$4: now also Q1.1; no longer Q1.2
Routing:
- net +6V5: track 82.8 -> 225.1 mm, vias 9 -> 18
- net +13V5: track 79.9 -> 207.1 mm
- net GND: track 971.3 -> 988.5 mm
- net +19V5: track 163.7 -> 157.0 mm
- net +12V: track 225.4 -> 230.5 mm
- net CTRL_CHARGING: track 127.1 -> 122.7 mm
- net N$19: track 6.60 -> 11.0 mm
- net VLOAD: track 43.6 -> 47.3 mm
- net +5V: track 375.4 -> 372.2 mm
- net N$17: track 127.7 -> 129.8 mm
- net N$24: track 2.68 -> 4.63 mm
- net +48V_B: track 75.7 -> 76.8 mm
- net N$22: track 2.24 -> 3.36 mm
- net +24V: track 179.1 -> 178.3 mm
- added copper zone on layer 1, net VBAT
- added copper zone on layer 1, net VLOAD
- added copper zone on layer 1, net VPWRSPLY
