File: board_sr/sr_controller_v1/sr_controller_v1_revC.sch (EAGLE design)
At the start: 74 parts, among them K1 PIN20X2, Q1 32kHz, Q3 IRF5210

Commit message: Publish sr_controller_v1_revC
Parts:
- removed C10, C12: C100nF, resistor:C-EUC0805
- removed C11, C13: C22pF, resistor:C-EUC0805
- removed C14: C100N, resistor:C-EUC0805K
- removed C7, C8: C100uF, resistor:CPOL-EU153CLV-0605
- removed C9: C4.7uF, resistor:C-EUC0805
- removed IC1: (no value), microbuilder:GSM_SIM900_LITERAL
- removed J1: (no value), SparkFun-Connectors:SIMHOLDERSIM
- removed K1: PIN20X2, FLYFISH:PIN20X2
- removed LED1, LED2: (no value), adafruit:LEDCHIPLED_0805
- removed Q3: IRF5210, transistor-power:PMOSFET_PTO220BV
- removed R18, R19: R22R, resistor:R-EU_R0805
- removed R23: R1K, resistor:R-EU_R0805
- removed R9: R20K, resistor:R-EU_R0805
- removed T2, T3, T4: (no value), transistor:MMBT2222ALT1-NPN-SOT23-BEC
- removed U$7: DCDCMODULE_SMALL, bontor:DCDCMODULE_SMALL
- removed U$9: TRANSFORMER, bontor:TRANSFORMER
- removed V_ACCU, V_LOAD, V_PWR_SPLY: (no value), con-ptr500:AK300/2
- removed V_SENSORS: (no value), con-ptr500:AK300/5
- removed X1: (no value), microbuilder:SMACONNECTOR
- added ADJ_VPWRSPLY, FROM_GREY_REG, FROM_LTC_REG, TO_GREY_REG, TO_LTC_REG, VBAT, VPWRSPLY: (no value), con-ptr500:AK300/2
- added B1: (no value), rectifier:RB1A
- added C2: C470uF, resistor:CPOL-EUE3.5-8
- added D1: 1N4004, diode:1N4004
- added F1, F2, F3: 5A, tigorcustom:BLADE_FUSE_HOLDER
- added FAN_A: 1X2-3.5MM, adafruit:1X2-3.5MM
- added IC3: LM741D, linear:LM741D
- added INDICATOR_CONN: (no value), con-lstb:MA03-2
- added J2, J3, J4, J5, J6, J7, J8, J9: WIRE_HOLE-14AWG, powercube:WIRE_HOLE-14AWG
- added OUT_+12V, OUT_+13V5, OUT_+19V5, OUT_+24V, OUT_+48V_A, OUT_+48V_B, OUT_+6V5: (no value), con-ptr500:AK500/2
- added PCB1: RASPBERRY_PI_B+_NO_MOUNT, tigorcustom:RASPBERRY_PI_B+_NO_MOUNT
- added Q2: BD140, transistor-power:BD140
- added R2, R4, R54: R10K, resistor:R-EU_R0805
- added R3, R34: R2K, resistor:R-EU_R0805
- added R53: R1K, resistor:R-EU_R0805
- added R55: R10K, ptc-ntc:NTC642-6
- added R57: R47R, resistor:R-EU_R0805
- added RPI_RESET: (no value), SparkFun-Electromechanical:TAC_SWITCHPTH
- added SJ1, SJ2, SJ4, SJ5: (no value), microbuilder:SOLDERJUMPER
- added SJ3: (no value), microbuilder:SOLDERJUMPERCLOSED
- added SJ6: (no value), microbuilder:SOLDERJUMPERREFLOW
- added TV16: TRANSFORMER, bontor:TRANSFORMER
- added U$10: DCDCMODULE, bontor:DCDCMODULE
- C3, C5: value C100N -> C100nF
- C4: value C1N -> C1nF
- C6: value C1N -> C1NF
- D2: value 18V -> 1N4004; device diode:ZENER-DIODEDO41Z10 -> diode:1N4004
- D3: value (none) -> 1N4728; device microbuilder:TVSARRAY_5LANE -> diode:1N4728
- R11: value R2K -> R1K
- R15: value R2K -> R10K
- R17: value R5K -> R5.1K
- R20: value R22R -> R1K
- R22: value R10K -> R5K
- R24, R26: value R1K -> R10K
- R27: value R120R -> R10K
- R29: value R2K -> R5.1K
- R32: value R100K -> R270K; device resistor:R-EU_0309/V -> resistor:R-EU_0309/10
- R33: value R2K -> R5K1; device resistor:R-EU_0309/V -> resistor:R-EU_0309/10
- R5: value R10K -> R150K
- R6: value R1K -> R100K
- R8: value R1K -> R220R
- U$3: value GND_CONNECT -> DCDCMODULE; device SparkFun-Passives:GND_CONNECT -> bontor:DCDCMODULE
- U$5: value FB0603 -> DCDCMODULE; device tigorcustom:L0603 -> bontor:DCDCMODULE
- U$6: value DCDCMODULE_SMALL -> DCDCMODULE; device bontor:DCDCMODULE_SMALL -> bontor:DCDCMODULE
Connections:
- net SENSOR_BUC renamed SENSOR_+48V_B
- net SENSOR_SCPC renamed SENSOR_+48V_A
- removed net CTRL_SIM_PWRKEY: K1.15, R27.1
- removed net N$11: D2.A, Q3.G, R5.2, R9.1
- removed net N$12: D2.C, Q3.S, R5.1, V_PWR_SPLY-2.KL
- removed net N$14: R9.2, T4.C
- removed net N$25: IC1.SIM_CLK, R19.1
- removed net N$27: LED1.C, T1.C
- removed net N$28: LED1.A, R23.2
- removed net N$29: LED2.C, T2.C
- removed net N$30: R21.2, R22.2, T1.B
- removed net N$31: LED2.A, R26.2
- removed net N$32: R24.2, R25.2, T2.B
- removed net N$33: R27.2, T3.B
- removed net SELECT_SENSOR: U$1.*10, U$8.S1
- removed net SENSOR_HI_1: R14.2, R15.1, U$8.1Y1
- removed net SENSOR_HI_2: R28.2, R29.1, U$8.1Y0
- removed net SENSOR_HUG_IDIR: U$1.A7, U$8.1Z
- removed net SENSOR_SCADA: R16.2, R17.1, U$1.A6
- removed net SIM_NETLIGHT: IC1.NETLIGHT, R24.1
- removed net SIM_PWRKEY: IC1.PWRKEY, T3.C
- removed net SIM_RX: IC1.RXD, K1.8
- removed net SIM_STATUS: IC1.STATUS, R21.1
- removed net SIM_TX: IC1.TXD, K1.10
- removed net USIM_CLK: D3.C3, J1.CLK, R19.2
- removed net USIM_DATA: D3.C1, J1.I/O, R20.2
- removed net USIM_RST: D3.C2, J1.RST, R18.2
- removed net USIM_VDD: C10.2, C11.2, C12.2, C13.2, D3.C4, IC1.SIM_VDD, J1.VCC
- removed net VIN: R10.1, U$6.VIN, U$7.VIN, V_SENSORS-1.KL
- new net +12V: D2.C, FAN_A.1, FROM_LTC_REG-2.KL, IC3.V+, OUT_+12V-1.KL, R16.1, R5.1, R54.1, U$5.VIN
- new net +13V5: OUT_+13V5-1.KL, R28.1, SJ5.2
- new net +19V5: FROM_LTC_REG-1.KL, OUT_+19V5-1.KL, R2.1, U$10.VIN
- new net +24V: FROM_GREY_REG-1.KL, OUT_+24V-1.KL, R4.1, TO_LTC_REG-1.KL, U$3.VIN, U$6.VIN
- new net +48V_A: F2.1, J6.P$1, J7.P$1, OUT_+48V_A-1.KL, R10.1
- new net +48V_B: F3.1, J8.P$1, J9.P$1, OUT_+48V_B-1.KL, R12.1
- new net +6V5: OUT_+6V5-1.KL, R14.1, SJ4.2
- new net ADJ_VOLTAGE: ADJ_VPWRSPLY-2.KL, R22.2
- new net INDC_HEALTH_BLUE: INDICATOR_CONN.3, PCB1.GPIO19, R26.2
- new net INDC_HEALTH_GREEN: INDICATOR_CONN.2, PCB1.GPIO20, R25.2
- new net INDC_HEALTH_RED: INDICATOR_CONN.1, PCB1.GPIO26, R24.2
- new net INDC_SPLY_OUTS: INDICATOR_CONN.4, PCB1.GPIO16, R27.2
- new net N$17: F1.1, TO_GREY_REG-2.KL
- new net N$39: IC3.OUT, R57.2
- new net N$40: Q2.B, R57.1
- new net N$7: U$8.1Y0, U$8.3Z
- new net N$8: SJ1.1, U$3.VOUT
- new net N$9: SJ2.1, U$6.VOUT
- new net RPI_RESET: PCB1.GPIO12, R53.2, RPI_RESET.1, RPI_RESET.2
- new net SEL_SENSOR_1: U$1.*11, U$8.S1
- new net SEL_SENSOR_2: U$1.12, U$8.S2
- new net SEL_SENSOR_3: U$1.13, U$8.S3
- new net SENSOR_+12V: R16.2, R17.1, U$8.3Y1
- new net SENSOR_+13V5: R28.2, R29.1, U$8.2Y0
- new net SENSOR_+19V5: R2.2, R3.1, U$8.2Y1
- new net SENSOR_+24V: R34.1, R4.2, U$1.A7
- new net SENSOR_+6V5: R14.2, R15.1, U$8.3Y0
- new net SENSOR_SPLY: U$1.A6, U$8.1Z
- new net VPWRSPLY: U$2.IP+@1, U$2.IP+@2, U$4.IP+@1, U$4.IP+@2, VPWRSPLY-2.KL
- net +3V3: now also INDICATOR_CONN.5, R24.1, R25.1, R27.1, R53.1, SJ2.2; no longer R23.1, U$5.P$2, U$7.VOUT
- net +5V: now also PCB1.5V0@1, PCB1.5V0@2, R21.2, SJ1.2; no longer K1.2, K1.4, U$6.VOUT
- net AGND: now also D3.A, SJ3.2, SJ6.1; no longer C14.1, U$3.AGND
- net ARDU_RX: now also PCB1.TXD0/GPIO14; no longer K1.35
- net ARDU_TX: now also PCB1.RXD0/GPIO15; no longer K1.37
- net CTRL_CHARGING: now also PCB1.GPIO18, R20.1; no longer K1.11, R6.1
- net DHT_DATA: now also U$1.*10; no longer U$1.12
- net GND: now also ADJ_VPWRSPLY-1.KL, FROM_GREY_REG-2.KL, IC3.V-, INDICATOR_CONN.6, OUT_+12V-2.KL, OUT_+13V5-2.KL, OUT_+19V5-2.KL, OUT_+24V-2.KL, OUT_+48V_A-2.KL, OUT_+48V_B-2.KL, OUT_+6V5-2.KL, PCB1.GND@1, PCB1.GND@2, PCB1.GND@3, Q2.C, R3.2, R34.2, R55.1, R6.2, RPI_RESET.3, RPI_RESET.4, SJ3.1, TO_GREY_REG-1.KL, TO_LTC_REG-2.KL, U$10.GNDI, U$10.GNDO, U$3.GNDI, U$3.GNDO, U$5.GNDI, U$5.GNDO, VBAT-1.KL, VPWRSPLY-1.KL; no longer C10.1, C11.1, C12.1, C13.1, C7.-, C8.-, C9.1, D3.A, IC1.GND@1, IC1.GND@10, IC1.GND@11, IC1.GND@12, IC1.GND@13, IC1.GND@14, IC1.GND@15, IC1.GND@2, IC1.GND@3, IC1.GND@4, IC1.GND@5, IC1.GND@6, IC1.GND@7, IC1.GND@8, IC1.GND@9, J1.GND, K1.14, K1.20, K1.25, K1.30, K1.34, K1.39, K1.6, K1.9, R22.1, R25.1, T2.E, T3.E, T4.E, U$3.DGND, U$7.GNDI, U$7.GNDO, V_ACCU-1.KL, V_LOAD-1.KL, V_PWR_SPLY-1.KL, X1.GND1, X1.GND2, X1.GND3, X1.GND4
- net N$13: now also SJ4.1, U$5.VOUT; no longer R6.2, T4.B
- net N$15: now also IC3.+IN, R54.2, R55.2; no longer Q3.D, U$4.IP+@1, U$4.IP+@2
- net N$18: now also IC3.-IN, R5.2, R6.1; no longer R14.1, V_SENSORS-3.KL
- net N$19: now also D1.A, R21.1, T1.C; no longer R28.1, V_SENSORS-4.KL
- net N$2: now also TV16.IB; no longer U$9.IB
- net N$20: now also D2.A, FAN_A.2, Q2.E; no longer R16.1, V_SENSORS-5.KL
- net N$21: now also B1.AC1, R33.2, TV16.OA; no longer IC1.RF_ANT, X1.ANT
- net N$22: now also R20.2, T1.B; no longer C7.+, C8.+, IC1.VBAT1, IC1.VBAT2, IC1.VBAT3, U$5.P$1
- net N$23: now also SJ5.1, U$10.VOUT; no longer C9.2, IC1.VRTC
- net N$24: now also D1.C, R22.1; no longer IC1.SIM_RST, R18.1
- net N$26: now also B1.-, C2.-, SJ6.2; no longer IC1.SIM_DATA, R20.1
- net N$3: now also Q1.1; no longer Q1.2
- net N$36: now also TV16.IA; no longer U$9.IA
- net N$38: now also B1.AC2, TV16.OB; no longer C14.2, U$9.OB
- net N$4: now also Q1.2; no longer Q1.1
- net N$6: now also U$8.1Y1, U$8.2Z; no longer R12.1, V_SENSORS-2.KL
- net RTC_SCL: now also PCB1.GPIO3/SCL1; no longer K1.5
- net RTC_SDA: now also PCB1.GPIO2/SDA1; no longer K1.3
- net SENSOR_IBAT: now also U$1.A0; no longer U$1.A2
- net SENSOR_ILOAD: now also U$1.A2; no longer U$1.A3
- net SENSOR_VAC: now also B1.+, C2.+, D3.C, U$1.A3; no longer R33.2, U$1.A0, U$9.OA
- net VBAT: now also J4.P$1, J5.P$1, VBAT-2.KL; no longer U$2.IP+@1, U$2.IP+@2, V_ACCU-2.KL
- net VLOAD: now also F1.2, F2.2, F3.2, J2.P$1, J3.P$1; no longer V_LOAD-2.KL
Other:
- note added: "Control_VPWRSPLY"
- note added: "Cooling_Fans"
- note added: "Indicator_LED"
- note added: "Sensor_IBAT"
- note added: "Sensor_ILOAD"
- note added: "Sensor_VAC"
- note added: "Sensor_VBAT"
- note added: "Supply_+12V_&_+19V5"
- note added: "Supply_+24V"
- note added: "Supply_+3V3_&_+5V"
- note added: "Supply_+48V"
- note added: "Supply_+6V5_&_+13V5"
- note added: "Supply_Outputs"
- note added: "Supply_Outputs_Sensor"
- note added: "v1"
- note removed: "CHARGING_&_SENSOR_IBAT"
- note removed: "Checked by:"
- note removed: "Drawn by:"
- note removed: "FLYFISH TECHNOLOGIES d.o.o."
- note removed: "Ivan Zilic"
- note removed: "SENSOR_ILOAD"
- note removed: "SENSOR_MODEMS"
- note removed: "SENSOR_VAC"
- note removed: "SENSOR_VBAT"
- note removed: "v0.1"
- moved on the sheet: BAT1, C1, C3, C4, C5, C6, Q1, R1, R10, R11, R12, R13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

Commit message: Update sr_controller_v1_revC
Parts:
- added FROM_LTC_REG_B: (no value), con-ptr500:AK300/2
- C6: value C1NF -> C1nF
- R33: value R5K1 -> R5.1K
- renumbered FROM_LTC_REG to FROM_LTC_REG_A
Connections:
- net +12V: now also FROM_LTC_REG_B-1.KL; no longer FROM_LTC_REG_A-2.KL
- net +13V5: now also FROM_LTC_REG_A-2.KL
- net +6V5: now also FROM_LTC_REG_B-2.KL
- net N$3: now also Q1.2; no longer Q1.1
- net N$4: now also Q1.1; no longer Q1.2
Other:
- note added: "Supply_+12V_&_+6V5"
- note added: "Supply_+19V5_&_+13V5"
- note removed: "Supply_+12V_&_+19V5"
- moved on the sheet: Q1
Changed lines of the file:
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@@
 <part name="AGND4" library="supply1" deviceset="AGND" device=""/>
 <part name="P+7" library="supply1" deviceset="+5V" device=""/>
-<part name="C6" library="resistor" deviceset="C-EU" device="C0805K" value="C1NF"/>
+<part name="C6" library="resistor" deviceset="C-EU" device="C0805K" value="C1nF"/>
 <part name="AGND5" library="supply1" deviceset="AGND" device=""/>
 <part name="R10" library="resistor" deviceset="R-EU_" device="R0805" value="R10K"/>
@@
 <part name="TV16" library="bontor" deviceset="TRANSFORMER" device=""/>
 <part name="R32" library="resistor" deviceset="R-EU_" device="0309/10" value="R270K"/>
-<part name="R33" library="resistor" deviceset="R-EU_" device="0309/10" value="R5K1"/>
+<part name="R33" library="resistor" deviceset="R-EU_" device="0309/10" value="R5.1K"/>
 <part name="R2" library="resistor" deviceset="R-EU_" device="R0805" value="R10K"/>
 <part name="R3" library="resistor" deviceset="R-EU_" device="R0805" value="R2K"/>
@@
 <part name="GND31" library="supply1" deviceset="GND" device=""/>
 <part name="FRAME2" library="frames" deviceset="FRAME_D_L" device=""/>
-<part name="FROM_LTC_REG" library="con-ptr500" deviceset="AK300/2" device=""/>
+<part name="FROM_LTC_REG_A" library="con-ptr500" deviceset="AK300/2" device=""/>
 <part name="F1" library="tigorcustom" deviceset="BLADE_FUSE_HOLDER" device="" value="5A"/>
 <part name="F2" library="tigorcustom" deviceset="BLADE_FUSE_HOLDER" device="" value="5A"/>
@@
 <part name="SJ6" library="microbuilder" deviceset="SOLDERJUMPER" device="REFLOW"/>
 <part name="AGND6" library="supply1" deviceset="AGND" device=""/>
+<part name="FROM_LTC_REG_B" library="con-ptr500" deviceset="AK300/2" device=""/>
 </parts>
 <sheets>
@@
 <text x="48.26" y="78.74" size="2.54" layer="98">Supply_+3V3_&amp;_+5V</text>
 <text x="154.94" y="78.74" size="2.54" layer="98">Supply_+6V5_&amp;_+13V5</text>
-<text x="241.3" y="78.74" size="2.54" layer="98">Supply_+12V_&amp;_+19V5</text>
+<text x="241.3" y="81.28" size="2.54" layer="98">Supply_+19V5_&amp;_+13V5</text>
 <text x="251.46" y="40.64" size="2.54" layer="98">Supply_+24V</text>
 <text x="299.72" y="78.74" size="2.54" layer="98">Supply_+48V</text>
@@
 <text x="53.34" y="190.5" size="2.54" layer="98">Control_VPWRSPLY</text>
 <text x="248.92" y="133.35" size="2.54" layer="98">Indicator_LED</text>
+<text x="241.3" y="76.2" size="2.54" layer="98">Supply_+12V_&amp;_+6V5</text>
 </plain>
 <instances>
@@
 <attribute name="VALUE" x="574.04" y="132.08" size="1.778" layer="96" rot="R180"/>
 </instance>
-<instance part="Q1" gate="G$1" x="523.24" y="121.92" rot="R270"/>
+<instance part="Q1" gate="G$1" x="523.24" y="121.92" rot="R90"/>
 <instance part="BAT1" gate="G$1" x="523.24" y="106.68" rot="R270"/>
 <instance part="GND9" gate="1" x="523.24" y="96.52"/>
@@
 <instance part="FRAME2" gate="G$1" x="431.8" y="0"/>
 <instance part="FRAME2" gate="G$2" x="762" y="0"/>
-<instance part="FROM_LTC_REG" gate="-1" x="265.43" y="63.5"/>
-<instance part="FROM_LTC_REG" gate="-2" x="265.43" y="59.69"/>
+<instance part="FROM_LTC_REG_A" gate="-1" x="265.43" y="63.5"/>
+<instance part="FROM_LTC_REG_A" gate="-2" x="265.43" y="59.69"/>
 <instance part="F1" gate="1" x="283.21" y="24.13"/>
 <instance part="F2" gate="1" x="312.42" y="60.96"/>
@@
 <instance part="SJ6" gate="1" x="96.52" y="287.02" rot="R90"/>
 <instance part="AGND6" gate="VR1" x="96.52" y="276.86"/>
+<instance part="FROM_LTC_REG_B" gate="-1" x="265.43" y="55.88"/>
+<instance part="FROM_LTC_REG_B" gate="-2" x="265.43" y="52.07"/>
 </instances>
 <busses>
@@
 <label x="35.56" y="231.14" size="0.8128" layer="95" ratio="10" xref="yes"/>
 </segment>
+<segment>
+<pinref part="FROM_LTC_REG_A" gate="-2" pin="KL"/>
+<wire x1="270.51" y1="59.69" x2="271.78" y2="59.69" width="0.1524" layer="91"/>
+<label x="271.78" y="59.69" size="0.8128" layer="95" ratio="10" xref="yes"/>
+</segment>
 </net>
 <net name="+6V5" class="0">
@@
 <label x="35.56" y="246.38" size="0.8128" layer="95" ratio="10" xref="yes"/>
 </segment>
+<segment>
+<pinref part="FROM_LTC_REG_B" gate="-2" pin="KL"/>
+<wire x1="270.51" y1="52.07" x2="271.78" y2="52.07" width="0.1524" layer="91"/>
+<label x="271.78" y="52.07" size="0.8128" layer="95" ratio="10" xref="yes"/>
+</segment>
 </net>
 <net name="+19V5" class="0">
@@
 </segment>
 <segment>
-<pinref part="FROM_LTC_REG" gate="-1" pin="KL"/>
+<pinref part="FROM_LTC_REG_A" gate="-1" pin="KL"/>
 <wire x1="270.51" y1="63.5" x2="271.78" y2="63.5" width="0.1524" layer="91"/>
 <label x="271.78" y="63.5" size="0.8128" layer="95" ratio="10" xref="yes"/>
@@
 </segment>
 <segment>
-<pinref part="FROM_LTC_REG" gate="-2" pin="KL"/>
-<wire x1="270.51" y1="59.69" x2="271.78" y2="59.69" width="0.1524" layer="91"/>
-<label x="271.78" y="59.69" size="0.8128" layer="95" ratio="10" xref="yes"/>
+<pinref part="FROM_LTC_REG_B" gate="-1" pin="KL"/>
+<wire x1="270.51" y1="55.88" x2="271.78" y2="55.88" width="0.1524" layer="91"/>
+<label x="271.78" y="55.88" size="0.8128" layer="95" ratio="10" xref="yes"/>
 </segment>
 </net>
@@
 </segment>
 </net>
-<net name="N$3" class="0">
-<segment>
-<pinref part="Q1" gate="G$1" pin="1"/>
-<pinref part="U1" gate="G$1" pin="X1"/>
-<wire x1="523.24" y1="124.46" x2="530.86" y2="124.46" width="0.1524" layer="91"/>
-</segment>
-</net>
-<net name="N$4" class="0">
-<segment>
-<pinref part="Q1" gate="G$1" pin="2"/>
-<pinref part="U1" gate="G$1" pin="X2"/>
-<wire x1="523.24" y1="119.38" x2="530.86" y2="119.38" width="0.1524" layer="91"/>
-</segment>
-</net>
 <net name="RPI_RESET" class="0">
 <segment>
@@
 </segment>
 </net>
+<net name="N$3" class="0">
+<segment>
+<pinref part="U1" gate="G$1" pin="X1"/>
+<pinref part="Q1" gate="G$1" pin="2"/>
+<wire x1="530.86" y1="124.46" x2="523.24" y2="124.46" width="0.1524" layer="91"/>
+</segment>
+</net>
+<net name="N$4" class="0">
+<segment>
+<pinref part="U1" gate="G$1" pin="X2"/>
+<pinref part="Q1" gate="G$1" pin="1"/>
+<wire x1="530.86" y1="119.38" x2="523.24" y2="119.38" width="0.1524" layer="91"/>
+</segment>
+</net>
