File: board_sr/sr_controller_v1/sr_controller_v1_revE.brd (EAGLE design)
At the start: 130 x 150 mm, 97 parts, among them IC3 LM741D, J2 WIRE_HOLE-14AWG, J3 WIRE_HOLE-14AWG, J4 WIRE_HOLE-14AWG, J5 WIRE_HOLE-14AWG, J6 WIRE_HOLE-14AWG, J7 WIRE_HOLE-14AWG, J8 WIRE_HOLE-14AWG, J9 WIRE_HOLE-14AWG, Q1 32kHz, Q2 BD140

Commit message: Urgent Update board_sr only
Commited & Pussed by Maula
Parts:
- removed FAN_A: 1X2-3.5MM, adafruit:1X2-3.5MM
- removed J2, J3, J4, J5, J6, J7, J8, J9: WIRE_HOLE-14AWG, powercube:WIRE_HOLE-14AWG
- removed SJ4, SJ5: (no value), microbuilder:SOLDERJUMPER_ARROW_NOPASTE
- removed U$10, U$5: DCDCMODULE, bontor:DCDCMODULE
- removed VBAT, VPWRSPLY: (no value), con-ptr500:AK300/2
- added FAN: (no value), microbuilder:HEADER_1X02
- added LED1: (no value), led:CHIP-LED0805
- added R18: R220R, resistor:R0805
- added R9: R10K, resistor:R0805
- added U$7: 74HC4053D, tigorcustom:SO16
- added VPWRSPLY&VBAT: (no value), con-ptr500:AK300/3
- OUT_+12V, OUT_+13V5, OUT_+19V5, OUT_+24V, OUT_+48V_A, OUT_+48V_B, OUT_+6V5: device con-ptr500:AK500/2 -> con-phoenix-508:MKDSN1,5/2-5,08
- moved SJ3 41.8 mm to (100.0, 145.5)
- moved C3 14.0 mm to (49.0, 115.8), flipped to the bottom, turned to 0 degrees
- moved U$8 13.0 mm to (106.0, 93.0)
- moved C6 12.0 mm to (36.5, 119.5), flipped to the bottom, turned to 180 degrees
- moved U$3 10.0 mm to (25.0, 82.0)
- moved C5 9.84 mm to (36.5, 121.5), flipped to the bottom, turned to 180 degrees
- moved C4 8.62 mm to (49.0, 117.8), flipped to the bottom, turned to 0 degrees
- moved R8 8.32 mm to (27.0, 114.5), flipped to the top, turned to 90 degrees
- moved D3 7.29 mm to (92.0, 147.0)
- moved U$4 6.02 mm to (37.0, 114.0), flipped to the bottom, turned to 0 degrees
- moved R7 5.59 mm to (29.0, 114.5), flipped to the top, turned to 270 degrees
- moved U$2 5.02 mm to (48.0, 123.2), flipped to the bottom, turned to 180 degrees
- moved SJ6 4.65 mm to (84.2, 145.5), turned to 90 degrees
- moved SJ2 3.40 mm to (73.5, 79.5), turned to 0 degrees
- moved SJ1 2.50 mm to (80.2, 100.5)
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Connections:
- net SENSOR_SPLY renamed SENSOR_SPLY_B
- removed net N$13: SJ4.1, U$5.VOUT
- removed net N$23: SJ5.1, U$10.VOUT
- removed net SEL_SENSOR_3: U$1.16, U$8.9
- new net N$11: U$7.13, U$7.15
- new net N$12: LED1.C, R53.1
- new net N$28: U$7.12, U$7.4
- new net SENSOR_SPLY_A: U$1.28, U$7.14
- new net SENSOR_VPWRSPLY: R18.1, R9.2, U$1.19
- net +12V: now also FAN.1, OUT_+12V.2; no longer FAN_A.1, OUT_+12V.1, U$5.VIN
- net +13V5: now also OUT_+13V5.2; no longer OUT_+13V5.1, SJ5.2
- net +19V5: now also OUT_+19V5.2; no longer OUT_+19V5.1, U$10.VIN
- net +24V: now also OUT_+24V.2; no longer OUT_+24V.1
- net +3V3: now also LED1.A; no longer R53.1
- net +48V_A: now also OUT_+48V_A.2; no longer J6.P$1, J7.P$1, OUT_+48V_A.1
- net +48V_B: now also OUT_+48V_B.2; no longer J8.P$1, J9.P$1, OUT_+48V_B.1
- net +5V: now also U$7.16
- net +6V5: now also OUT_+6V5.2; no longer OUT_+6V5.1, SJ4.2
- net GND: now also OUT_+12V.1, OUT_+13V5.1, OUT_+19V5.1, OUT_+24V.1, OUT_+48V_A.1, OUT_+48V_B.1, OUT_+6V5.1, R18.2, U$7.6, U$7.7, U$7.8, VPWRSPLY&VBAT.1; no longer OUT_+12V.2, OUT_+13V5.2, OUT_+19V5.2, OUT_+24V.2, OUT_+48V_A.2, OUT_+48V_B.2, OUT_+6V5.2, U$10.GND#0, U$10.GND#1, U$5.GND#0, U$5.GND#1, VBAT.1, VPWRSPLY.1
- net N$20: now also FAN.2; no longer FAN_A.2
- net SEL_SENSOR_1: now also U$7.11
- net SEL_SENSOR_2: now also U$7.10, U$7.9, U$8.9
- net SENSOR_+24V: now also U$7.5; no longer U$1.28
- net SENSOR_+48V_A: now also U$7.2; no longer U$1.26
- net SENSOR_+48V_B: now also U$7.3; no longer U$1.25
- net SENSOR_IBAT: now also U$1.18; no longer U$1.17
- net SENSOR_ILOAD: now also U$1.17; no longer U$1.19
- net SENSOR_VBAT: now also U$7.1; no longer U$1.18
- net VBAT: now also VPWRSPLY&VBAT.3; no longer J4.P$1, J5.P$1, VBAT.2
- net VLOAD: no longer J2.P$1, J3.P$1
- net VPWRSPLY: now also R9.1, VPWRSPLY&VBAT.2; no longer VPWRSPLY.2
Routing:
- net SENSOR_VPWRSPLY: track 0.00 -> 114.0 mm
- net +13V5: track 209.4 -> 142.7 mm, vias 9 -> 0
- net +6V5: track 225.1 -> 174.5 mm, vias 18 -> 9
- net +5V: track 366.7 -> 328.0 mm, vias 10 -> 7
- net GND: track 987.3 -> 949.1 mm, vias 3 -> 11
- net +3V3: track 222.2 -> 251.7 mm, vias 4 -> 12
- net AGND: track 82.2 -> 108.2 mm, vias 2 -> 4
- net SENSOR_+48V_B: track 89.3 -> 114.7 mm
- net SEL_SENSOR_3: track 25.2 -> 0.00 mm
- net VPWRSPLY: track 24.5 -> 49.8 mm
- net SENSOR_+48V_A: track 80.8 -> 100.3 mm
- net SENSOR_VBAT: track 97.4 -> 78.8 mm
- net SENSOR_VAC: track 56.0 -> 74.7 mm
- net SEL_SENSOR_2: track 22.0 -> 39.9 mm, vias 0 -> 2
- net +24V: track 178.3 -> 195.1 mm
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- added copper zone on layer 16, net VLOAD
- removed copper zone on layer 1, net VBAT
- removed copper zone on layer 1, net VLOAD
- removed copper zone on layer 1, net VPWRSPLY
Other:
- board text added: "sr_controller_v1_revE"
- board text removed: "J2"
- board text removed: "J3"
- board text removed: "J4"
- board text removed: "J5"
- board text removed: "J6"
- board text removed: "J7"
- board text removed: "J8"
- board text removed: "J9"
