File: board_sr/sr_controller_v1/sr_controller_v1_revE.sch (EAGLE design)
At the start: 97 parts, among them IC3 LM741D, J2 WIRE_HOLE-14AWG, J3 WIRE_HOLE-14AWG, J4 WIRE_HOLE-14AWG, J5 WIRE_HOLE-14AWG, J6 WIRE_HOLE-14AWG, J7 WIRE_HOLE-14AWG, J8 WIRE_HOLE-14AWG, J9 WIRE_HOLE-14AWG, Q1 32kHz, Q2 BD140

Commit message: Urgent Update board_sr only
Commited & Pussed by Maula
Parts:
- removed FAN_A: 1X2-3.5MM, adafruit:1X2-3.5MM
- removed J2, J3, J4, J5, J6, J7, J8, J9: WIRE_HOLE-14AWG, powercube:WIRE_HOLE-14AWG
- removed SJ4, SJ5: (no value), microbuilder:SOLDERJUMPER
- removed U$10, U$5: DCDCMODULE, bontor:DCDCMODULE
- removed VBAT, VPWRSPLY: (no value), con-ptr500:AK300/2
- added FAN: (no value), microbuilder:HEADER_1X02
- added LED1: (no value), led:LEDCHIP-LED0805
- added R18: R220R, resistor:R-EU_R0805
- added R9: R10K, resistor:R-EU_R0805
- added U$7: 74HC4053D, tigorcustom:74HC4053D
- added VPWRSPLY&VBAT: (no value), con-ptr500:AK300/3
- OUT_+12V, OUT_+13V5, OUT_+19V5, OUT_+24V, OUT_+48V_A, OUT_+48V_B, OUT_+6V5: value (none) -> MKDSN1,5/2-5,08; device con-ptr500:AK500/2 -> con-phoenix-508:MKDSN1,5/2-5,08
Connections:
- net SENSOR_SPLY renamed SENSOR_SPLY_B
- removed net N$13: SJ4.1, U$5.VOUT
- removed net N$23: SJ5.1, U$10.VOUT
- removed net SEL_SENSOR_3: U$1.13, U$8.S3
- new net N$11: U$7.1Y1, U$7.2Z
- new net N$12: LED1.C, R53.1
- new net N$28: U$7.1Y0, U$7.3Z
- new net SENSOR_SPLY_A: U$1.A7, U$7.1Z
- new net SENSOR_VPWRSPLY: R18.1, R9.2, U$1.A2
- net +12V: now also FAN.1, OUT_+12V-2.KL; no longer FAN_A.1, OUT_+12V-1.KL, U$5.VIN
- net +13V5: now also OUT_+13V5-2.KL; no longer OUT_+13V5-1.KL, SJ5.2
- net +19V5: now also OUT_+19V5-2.KL; no longer OUT_+19V5-1.KL, U$10.VIN
- net +24V: now also OUT_+24V-2.KL; no longer OUT_+24V-1.KL
- net +3V3: now also LED1.A; no longer R53.1
- net +48V_A: now also OUT_+48V_A-2.KL; no longer J6.P$1, J7.P$1, OUT_+48V_A-1.KL
- net +48V_B: now also OUT_+48V_B-2.KL; no longer J8.P$1, J9.P$1, OUT_+48V_B-1.KL
- net +5V: now also U$7.VCC
- net +6V5: now also OUT_+6V5-2.KL; no longer OUT_+6V5-1.KL, SJ4.2
- net GND: now also OUT_+12V-1.KL, OUT_+13V5-1.KL, OUT_+19V5-1.KL, OUT_+24V-1.KL, OUT_+48V_A-1.KL, OUT_+48V_B-1.KL, OUT_+6V5-1.KL, R18.2, U$7./E, U$7.GND, U$7.VEE, VPWRSPLY&VBAT-1.KL; no longer OUT_+12V-2.KL, OUT_+13V5-2.KL, OUT_+19V5-2.KL, OUT_+24V-2.KL, OUT_+48V_A-2.KL, OUT_+48V_B-2.KL, OUT_+6V5-2.KL, U$10.GNDI, U$10.GNDO, U$5.GNDI, U$5.GNDO, VBAT-1.KL, VPWRSPLY-1.KL
- net N$20: now also FAN.2; no longer FAN_A.2
- net SEL_SENSOR_1: now also U$7.S1
- net SEL_SENSOR_2: now also U$7.S2, U$7.S3, U$8.S3
- net SENSOR_+24V: now also U$7.3Y0; no longer U$1.A7
- net SENSOR_+48V_A: now also U$7.2Y0; no longer U$1.A5
- net SENSOR_+48V_B: now also U$7.3Y1; no longer U$1.A4
- net SENSOR_IBAT: now also U$1.A1; no longer U$1.A0
- net SENSOR_ILOAD: now also U$1.A0; no longer U$1.A2
- net SENSOR_VBAT: now also U$7.2Y1; no longer U$1.A1
- net VBAT: now also VPWRSPLY&VBAT-3.KL; no longer J4.P$1, J5.P$1, VBAT-2.KL
- net VLOAD: no longer J2.P$1, J3.P$1
- net VPWRSPLY: now also R9.1, VPWRSPLY&VBAT-2.KL; no longer VPWRSPLY-2.KL
Other:
- note added: "Sensor_VPWRSPLY"
- note removed: "Supply_+6V5_&_+13V5"
- moved on the sheet: C3, C4, OUT_+12V-1, OUT_+12V-2, OUT_+13V5-1, OUT_+13V5-2, OUT_+19V5-1, OUT_+19V5-2, OUT_+24V-1, OUT_+24V-2, OUT_+48V_A-1, OUT_+48V_A-2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
